File: board/esp32_board/esp32_board.kicad_pcb (KiCad board)
At the start: 2 copper layers, 0 parts

Commit message: feat: Updated presentation and board
Parts:
- added J1: Screw_Terminal_01x19, Connector_PinHeader_2.54mm:PinHeader_1x19_P2.54mm_Vertical, F.Cu at (191.0, 74.5)
- added J2: Screw_Terminal_01x19, Connector_PinHeader_2.54mm:PinHeader_1x19_P2.54mm_Vertical, F.Cu at (103.5, 73.5)
- added U1: ESP32-DevKitC, PCM_Espressif:ESP32-DevKitC, F.Cu at (135.2, 74.5)
