File: board/esp32_board/esp32_board.kicad_sch (KiCad schematic)
At the start: 14 parts, among them J1 Screw_Terminal_01x19, J2 Screw_Terminal_01x19, J3 Conn_01x19_Socket, J4 Conn_01x19_Pin, J5 Conn_01x19_Socket, J6 Conn_01x19_Pin, U1 ESP32-DevKitC

Commit message: feat: Updated docs and board
Other:
- title: (none) -> Принципиальная схема
- moved on the sheet: J1, J2, J3, J4, J5, J6, R1, R2, U1, compass1, gps1, relay1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

Commit message: feat: Updated docs
Connections:
- net GND: now also relay3.4 (GND)
- net SIG: now reaches relay3.1 (SIG)
- net SIG: now also relay2.6 (1NC)
- net VCC: now reaches relay3.3 (VCC)
- net VCC: now also relay2.5 (1COM)
Other:
- moved on the sheet: J1, J5, J6, compass1, gps1

Commit message: feat: Final board version and updated docs
Parts:
- J1, J2, J3, J5: footprint Connector_PinHeader_2.54mm:PinHeader_1x19_P2.54mm_Vertical -> slon_modules:PinHeader_1x19_P2.54mm_Vertical
- J4, J6: footprint Connector_PinSocket_2.54mm:PinSocket_1x19_P2.54mm_Vertical -> slon_modules:PinHeader_1x19_P2.54mm_Vertical
Changed lines of the file:
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@@
 			)
 		)
-		(property "Footprint" "Connector_PinSocket_2.54mm:PinSocket_1x19_P2.54mm_Vertical"
+		(property "Footprint" "slon_modules:PinHeader_1x19_P2.54mm_Vertical"
 			(at 69.85 95.25 0)
 			(effects
@@
 			)
 		)
-		(property "Footprint" "Connector_PinHeader_2.54mm:PinHeader_1x19_P2.54mm_Vertical"
+		(property "Footprint" "slon_modules:PinHeader_1x19_P2.54mm_Vertical"
 			(at 104.14 161.29 0)
 			(effects
@@
 			)
 		)
-		(property "Footprint" "Connector_PinHeader_2.54mm:PinHeader_1x19_P2.54mm_Vertical"
+		(property "Footprint" "slon_modules:PinHeader_1x19_P2.54mm_Vertical"
 			(at 54.61 161.29 0)
 			(effects
@@
 			)
 		)
-		(property "Footprint" "Connector_PinHeader_2.54mm:PinHeader_1x19_P2.54mm_Vertical"
+		(property "Footprint" "slon_modules:PinHeader_1x19_P2.54mm_Vertical"
 			(at 95.25 95.25 0)
 			(effects
@@
 			)
 		)
-		(property "Footprint" "Connector_PinSocket_2.54mm:PinSocket_1x19_P2.54mm_Vertical"
+		(property "Footprint" "slon_modules:PinHeader_1x19_P2.54mm_Vertical"
 			(at 80.01 161.29 0)
 			(effects
@@
 			)
 		)
-		(property "Footprint" "Connector_PinHeader_2.54mm:PinHeader_1x19_P2.54mm_Vertical"
+		(property "Footprint" "slon_modules:PinHeader_1x19_P2.54mm_Vertical"
 			(at 45.72 95.25 0)
 			(effects
